File: hardware/sensor_board.brd (EAGLE design)
At the start: 50 x 17 mm, 12 parts, among them X5 i2c

Commit message: pcb verified
Parts:
- removed C7: 100nF, rcl:C0805
Connections:
- net +3V3: no longer C7.2
- net GND: no longer C7.1
Routing:
- net +3V3: track 51.0 -> 49.9 mm
- net GND: track 41.8 -> 42.4 mm
Changed lines of the file:
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@@
 <wire x1="-0.01" y1="17" x2="0" y2="0" width="0.4064" layer="20"/>
 <text x="30.2" y="1.7" size="1.01" layer="109" font="vector" ratio="15" rot="MR0"></text>
-<hole x="47.51" y="14.5" drill="3.2"/>
+<hole x="47.5" y="14.5" drill="3.2"/>
 <rectangle x1="19.7" y1="6.5" x2="21.2" y2="8" layer="30"/>
 <text x="34.46" y="15.45" size="1.016" layer="1" font="vector" ratio="15">1</text>
@@
 <rectangle x1="17.8" y1="5.1" x2="21.8" y2="9.4" layer="30"/>
 <text x="33.08" y="12.01" size="0.8128" layer="108" font="vector" ratio="15">i2c</text>
-<hole x="47.47" y="2.65" drill="3.2"/>
-<hole x="43.1" y="12.38" drill="3.2"/>
-<hole x="43.11" y="3.89" drill="3.2"/>
+<hole x="47.5" y="2.5" drill="3.2"/>
+<hole x="43" y="13" drill="3.2"/>
+<hole x="43" y="4" drill="3.2"/>
 <hole x="4.79" y="3.19" drill="2"/>
 <hole x="18.53" y="8.45" drill="2"/>
@@
 <element name="U$7" library="SparkFun" package="OSHW-LOGO-M" value="OSHW-LOGOM" x="2.96" y="13.81"/>
 <element name="X5" library="Simplex-Connectors" package="0530480401" value="i2c" x="34.08" y="6.38" rot="R90"/>
-<element name="C7" library="rcl" package="C0805" value="100nF" x="31.81" y="3.44" rot="R90"/>
 <element name="C15" library="rcl" package="C1206" value="10uF" x="29.77" y="3.42" rot="R270"/>
 <element name="R5" library="rcl" package="R0805W" value="330" x="28.66" y="9.08" rot="R180"/>
@@
 <contactref element="X5" pad="1"/>
 <contactref element="C15" pad="2"/>
-<contactref element="C7" pad="1"/>
 <contactref element="U$1" pad="1"/>
 <contactref element="C1" pad="1"/>
 <contactref element="C2" pad="1"/>
 <wire x1="25.78" y1="0.91" x2="14.8" y2="0.91" width="0.6096" layer="1"/>
-<wire x1="14.8" y1="0.91" x2="11.43" y2="0.91" width="0.6096" layer="1"/>
-<wire x1="11.43" y1="0.91" x2="8.685" y2="3.655" width="0.6096" layer="1"/>
-<wire x1="8.685" y1="3.655" x2="7.447" y2="3.655" width="0.6096" layer="1"/>
 <wire x1="14.75" y1="0.96" x2="14.8" y2="0.91" width="0.6096" layer="1"/>
 <wire x1="24.45" y1="12.51" x2="24.47" y2="12.53" width="0.6096" layer="1"/>
-<wire x1="5.47" y1="10.82" x2="5.47" y2="11.94" width="0.4064" layer="1"/>
-<wire x1="5.47" y1="11.94" x2="5.86" y2="12.33" width="0.4064" layer="1"/>
-<wire x1="5.86" y1="12.33" x2="24.27" y2="12.33" width="0.4064" layer="1"/>
 <wire x1="24.27" y1="12.33" x2="24.47" y2="12.53" width="0.4064" layer="1"/>
 <contactref element="U$2" pad="P$1"/>
@@
 <wire x1="14.71" y1="2.724" x2="14.71" y2="1" width="0.6096" layer="1"/>
 <wire x1="14.71" y1="1" x2="14.75" y2="0.96" width="0.6096" layer="1"/>
+<wire x1="14.71" y1="1" x2="12.055" y2="3.655" width="0.6096" layer="1"/>
+<wire x1="12.055" y1="3.655" x2="7.447" y2="3.655" width="0.6096" layer="1"/>
+<wire x1="5.47" y1="10.82" x2="5.47" y2="11.81" width="0.6096" layer="1"/>
+<wire x1="5.47" y1="11.81" x2="5.96" y2="12.3" width="0.6096" layer="1"/>
+<wire x1="5.96" y1="12.3" x2="11.53" y2="12.3" width="0.6096" layer="1"/>
+<wire x1="11.53" y1="12.3" x2="12.54" y2="11.29" width="0.6096" layer="1"/>
+<wire x1="12.54" y1="11.29" x2="24.66" y2="11.29" width="0.6096" layer="1"/>
+<wire x1="24.71" y1="11.29" x2="24.66" y2="11.29" width="0.6096" layer="1"/>
 </signal>
 <signal name="+3V3">
@@
 <contactref element="R13" pad="2"/>
 <contactref element="C15" pad="1"/>
-<contactref element="C7" pad="2"/>
 <contactref element="U$1" pad="4"/>
 <contactref element="C1" pad="2"/>
 <contactref element="C2" pad="2"/>
 <wire x1="34.08" y1="7.63" x2="33.47" y2="7.63" width="0.6096" layer="1"/>
-<wire x1="33.47" y1="7.63" x2="32.41" y2="6.57" width="0.6096" layer="1"/>
-<wire x1="32.41" y1="6.57" x2="32.41" y2="4.99" width="0.6096" layer="1"/>
-<wire x1="32.41" y1="4.99" x2="31.81" y2="4.39" width="0.6096" layer="1"/>
-<wire x1="31.81" y1="4.39" x2="31.54" y2="4.66" width="0.6096" layer="1"/>
-<wire x1="31.54" y1="4.66" x2="29.79" y2="4.66" width="0.6096" layer="1"/>
 <wire x1="29.79" y1="4.66" x2="27.63" y2="4.66" width="0.6096" layer="1"/>
 <wire x1="29.77" y1="4.82" x2="29.79" y2="4.8" width="0.6096" layer="1"/>
@@
 <wire x1="17.24" y1="2.724" x2="17.24" y2="4.51" width="0.6096" layer="1"/>
 <wire x1="17.24" y1="4.51" x2="17.39" y2="4.66" width="0.6096" layer="1"/>
+<wire x1="33.47" y1="7.63" x2="30.5" y2="4.66" width="0.6096" layer="1"/>
+<wire x1="30.5" y1="4.66" x2="29.79" y2="4.66" width="0.6096" layer="1"/>
 </signal>
 <signal name="SCL_H">

Commit message: board ready
Changed lines of the file:
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@@
 <layers>
 <layer number="1" name="Top" color="4" fill="1" visible="yes" active="yes"/>
-<layer number="2" name="Route2" color="1" fill="3" visible="yes" active="yes"/>
+<layer number="2" name="Route2" color="1" fill="3" visible="no" active="no"/>
 <layer number="3" name="Route3" color="4" fill="3" visible="no" active="no"/>
 <layer number="14" name="Route14" color="1" fill="6" visible="no" active="no"/>
-<layer number="15" name="Route15" color="4" fill="6" visible="yes" active="yes"/>
+<layer number="15" name="Route15" color="4" fill="6" visible="no" active="no"/>
 <layer number="16" name="Bottom" color="1" fill="1" visible="yes" active="yes"/>
 <layer number="17" name="Pads" color="2" fill="1" visible="yes" active="yes"/>
@@
 <hole x="47.5" y="14.5" drill="3.2"/>
 <rectangle x1="19.7" y1="6.5" x2="21.2" y2="8" layer="30"/>
-<text x="34.46" y="15.45" size="1.016" layer="1" font="vector" ratio="15">1</text>
-<text x="36.25" y="16.49" size="1.016" layer="16" font="vector" ratio="15" rot="R180">2</text>
+<text x="34.22" y="15.19" size="1.016" layer="1" font="vector" ratio="15">1</text>
+<text x="35.45" y="15.17" size="1.016" layer="16" font="vector" ratio="15">2</text>
 <wire x1="4.7" y1="41.06" x2="7.5" y2="41.06" width="1.6764" layer="42"/>
 <rectangle x1="17.8" y1="5.1" x2="21.8" y2="9.4" layer="30"/>
@@
 </class>
 </classes>
-<designrules name="SeeedStudio_DRU_no_angle_20130527">
+<designrules name="seeed_2-layer_20140221">
 <description language="de">&lt;b&gt;EAGLE Design Rules&lt;/b&gt;
 &lt;p&gt;
@@
 <description language="zh">&lt;b&gt;Seeed Studio EAGLE Design Rules&lt;/b&gt;
 </description>
-<param name="layerSetup" value="(1*2*15*16)"/>
+<param name="layerSetup" value="(1*16)"/>
 <param name="mtCopper" value="0.035mm 0.0175mm 0.035mm 0.035mm 0.035mm 0.035mm 0.035mm 0.035mm 0.035mm 0.035mm 0.035mm 0.035mm 0.035mm 0.035mm 0.0175mm 0.035mm"/>
-<param name="mtIsolate" value="0.2mm 1.1mm 0.2mm 0.15mm 0.2mm 0.15mm 0.2mm 0.15mm 0.2mm 0.15mm 0.2mm 0.15mm 0.2mm 0.15mm 0.2mm"/>
+<param name="mtIsolate" value="1.5mm 1.1mm 0.2mm 0.15mm 0.2mm 0.15mm 0.2mm 0.15mm 0.2mm 0.15mm 0.2mm 0.15mm 0.2mm 0.15mm 0.2mm"/>
 <param name="mdWireWire" value="6mil"/>
 <param name="mdWirePad" value="6mil"/>
@@
 <param name="rlMinPadTop" value="6mil"/>
 <param name="rlMaxPadTop" value="20mil"/>
-<param name="rlMinPadInner" value="6mil"/>
+<param name="rlMinPadInner" value="10mil"/>
 <param name="rlMaxPadInner" value="20mil"/>
 <param name="rlMinPadBottom" value="6mil"/>
@@
 <param name="mlMinCreamFrame" value="0mil"/>
 <param name="mlMaxCreamFrame" value="0mil"/>
-<param name="mlViaStopLimit" value="25mil"/>
+<param name="mlViaStopLimit" value="100mil"/>
 <param name="srRoundness" value="0"/>
 <param name="srMinRoundness" value="0mil"/>
