File: hardware/sensor_board.sch (EAGLE design)
At the start: 88 parts, among them IC1 SIM900, IC2 DS3231, J2 U.FL, Q2 PMBF170, Q3 PMBF170, Q4 si2305cd, Q5 si2305cd, T1 BC846, T2 BC846, T4 BC846, U1 SPX5205 3v3, U3 TC1014 2V8, X1 prog, X2 bat, X4 ts, X5 i2c, X6 pwr, Y1 32768Hz CFPX-217 12.5pF

Commit message: add sensor board
Parts:
- removed C10: 470nF, rcl:C-EUC0805
- removed C12: 4u7, rcl:C-EUC0805
- removed C13, C17, C18, C22, C25, C26, C29, C5, C6, C8, C9: 100nF, rcl:C-EUC0805
- removed C14, C23, C24: 22pF, rcl:C-EUC0805
- removed C16, C20, C21: 100uF, rcl:C-EUC1206
- removed C27, C28: 4u7, rcl:C-EUC1206
- removed C3: 10uF, rcl:C-EUC0805
- removed C30: 10uF, rcl:C-EUC1206
- removed C32, C4: 1uF, rcl:C-EUC0805
- removed G1: HU2032-LF, Simplex-Battery:HU2032-LF
- removed IC1: SIM900, Simplex-ICs:SIM900
- removed IC2: DS3231, Simplex-ICs:DS3231
- removed J2: U.FL, SparkFun-Connectors:U.FL
- removed LED1: green, led:LEDCHIPLED_0805
- removed Q2, Q3: PMBF170, Simplex-DiscreteSemi:MOSFET-NCHANNEL_SOT23-3
- removed Q4, Q5: si2305cd, Simplex-DiscreteSemi:MOSFET-PCHANNELSMD_POWER
- removed R1, R10, R2, R23: 10k, rcl:R-EU_R0805W
- removed R11: 3k, rcl:R-EU_R0805W
- removed R12: 100K, rcl:R-EU_R0805W
- removed R14: DNP 10k th, rcl:R-EU_R0805W
- removed R15: 1k1, rcl:R-EU_R0805W
- removed R16, R20: 4k7, rcl:R-EU_R0805W
- removed R18, R34, R35: 47k, rcl:R-EU_R0805W
- removed R21, R6: 100k, rcl:R-EU_R0805W
- removed R22, R3: 2M, rcl:R-EU_R0805W
- removed R24: 620K, rcl:R-EU_R0805W
- removed R4: 1M3, rcl:R-EU_R0805W
- removed R9: 220K, rcl:R-EU_R0805W
- removed T1, T2, T4: BC846, transistor:BC846
- removed TP1, TP101, TP102, TP2, TP3, TP4, TP5, TP6, TP7: TPTP12R, testpad:TPTP12R
- removed U$10: bead, Simplex-rlc:INDUCTOR
- removed U$17: FM24V, Simplex-ICs:FM24V
- removed U$18: 22, Simplex-rlc:RES_ARR
- removed U$3: SIM_MOLEX_7880-0001, Simplex-Connectors:SIM_MOLEX_7880-0001
- removed U$6: BQ24072, Simplex-ICs:BQ24072
- removed U$8: SMF05C, Simplex-DiscreteSemi:SMF05C
- removed U$9: RESETTABLE_0805, Simplex-Fuses:RESETTABLE_0805
- removed U1: SPX5205 3v3, SparkFun:V_REG_LDOSMD
- removed U3: TC1014 2V8, SparkFun:V_REG_LDOSMD
- removed X1: prog, Simplex-Connectors:MOLEX_6VERTICAL
- removed X2: bat, Simplex-Connectors:MOLEX_2HORIZONTAL
- removed X4: ts, Simplex-Connectors:MOLEX_2HORIZONTAL
- removed X6: pwr, Simplex-Connectors:MOLEX_4HORIZONTAL
- removed Y1: 32768Hz CFPX-217 12.5pF, Simplex-FreqCtrl:CRYSTAL3.2X1.5
- added C15: 10uF, rcl:C-EUC1206
- added R5, R7: 330, rcl:R-EU_R0805W
- added R8: 10k, rcl:R-EU_R0805W
- C7: value 10uF -> 100nF; device rcl:C-EUC1206 -> rcl:C-EUC0805
- R13: value 4k7 -> 10k
- U$1: value MSP430F5510 -> SHT1XSMD; device TI_MSP430_v16:F55[0/1]X---PT48 -> SparkFun-Sensors:SHT1XSMD
- U$2: value 470 -> HONEYWELL_HSC; device Simplex-rlc:RES_ARR -> Simplex-ICs:HONEYWELL_HSC
Connections:
- removed net 2V8: C17.2, C29.1, C30.1, C8.2, C9.2, Q5.S, R34.2, R9.1, TP102.TP, U$1.11, U$1.28, U$1.7, U3.OUT, X1.3
- removed net 2V8_SW: C25.1, C5.1, IC2.VCC, Q2.G, Q3.G, Q5.D, R1.1, R13.2, R16.2, U$17.VCC
- removed net 5V_IN: R22.1, U$6G$1.IN, U$9.P$2
- removed net BAT: C27.1, R3.1, U$6G$1.BAT, X2.1
- removed net BAT_DIV: C2.1, R3.2, R4.1, U$1.4
- removed net CE: U$1.45, U$6G$1.CE, X6.1
- removed net CHG: U$1.46, U$6G$1.CHG
- removed net CTS: IC1G$1.CTS, U$1.18
- removed net DTR: IC1G$1.DTR, U$1.20
- removed net GPRS_PWRKEY: R20.2, U$1.29
- removed net GPRS_RX: IC1G$1.RXD, TP4.TP, U$2.7
- removed net GPRS_TX: IC1G$1.TXD, TP5.TP, U$2.8
- removed net GPRS_VBAT: R23.1, U$1.30
- removed net I2C_EN: R12.1, U$1.1, U1.EN
- removed net N$1: U$1.32, U$2.3
- removed net N$10: U$1.34, U$2.1
- removed net N$14: Q5.G, R9.2, T4.C
- removed net N$15: R12.2, T4.B
- removed net N$17: IC1G$1.SIM_DATA, U$18.8
- removed net N$18: IC1G$1.SIM_CLK, U$18.7
- removed net N$19: IC1G$1.SIM_RST, U$18.6
- removed net N$2: C4.1, U1.BP
- removed net N$25: C24.1, U$1.9, Y1.1
- removed net N$26: C23.1, U$1.8, Y1.2
- removed net N$27: R11.1, U$6G$1.ISET
- removed net N$3: U$1.31, U$2.4
- removed net N$33: R15.1, U$6G$1.ILIM
- removed net N$4: U$1.33, U$2.2
- removed net N$45: R18.2, R20.1, T2.B
- removed net N$46: IC1G$1.RF_ANT, J2.SIGNAL
- removed net N$48: C22.2, Q4.G, R21.1, T1.C
- removed net N$49: C22.1, Q4.D, U$10.1
- removed net N$5: G1.+, IC2.VBAT
- removed net N$50: C32.1, U3.BP
- removed net N$6: C10.1, U$1.13
- removed net N$7: R23.2, T1.B
- removed net N$8: LED1.C, R6.1
- removed net N$9: IC2.32KHZ, R1.2
- removed net PWRKEY: IC1G$1.PWRKEY, T2.C
- removed net RAW_DIV: C18.1, R22.2, R24.1, U$1.3
- removed net RI: IC1G$1.RI, U$1.19
- removed net RST: R34.1, U$1.48, X1.5
- removed net RTS: IC1G$1.RTS, U$1.17
- removed net SCL_L: IC2.SCL, Q2.S, R13.1, U$1.35, U$17.SCL
- removed net SDA_L: IC2.SDA, Q3.S, R16.1, U$1.36, U$17.SDA
- removed net SIMLOCK_CLK: U$18.2, U$3.CLK, U$8.CATODE3
- removed net SIMLOCK_IO: C14.2, U$18.1, U$3.IO, U$8.CATODE4
- removed net SIMLOCK_RST: U$18.3, U$3.RST, U$8.CATODE5
- removed net SIM_VCC: C13.2, IC1G$1.SIM_VDD, U$3.VCC, U$8.CATODE2
- removed net STATUS: LED1.A, TP6.TP, U$1.2
- removed net TEST: R35.1, U$1.47, X1.4
- removed net TS: R14.1, U$6G$1.TS, X4.2
- removed net UART_RX: TP2.TP, U$2.5, X1.2
- removed net UART_TX: TP3.TP, U$2.6, X1.1
- removed net VBAT: C16.1, C20.1, C21.1, C26.1, U$10.2
- removed net VIN: C28.1, C3.1, C6.1, Q4.S, R21.2, U$6G$1.EN2, U$6G$1.OUT, U1.IN, U3.EN, U3.IN
- removed net VRAW: U$9.P$1, X6.2, X6.3
- removed net VRTC: C12.2, IC1G$1.VRTC
- new net SCL: R5.2, R8.1, U$1.SCK, U$2.SCL
- new net SDA: R13.1, R7.2, U$1.DATA, U$2.SDA
- net +3V3: now also C1.2, C15.1, C2.2, C7.2, R13.2, R8.2, U$1.VDD, U$2.VCC; no longer C1.1, C7.1, R10.2, R2.2, TP7.TP, U1.OUT
- net GND: now also C1.1, C15.2, C2.1, C7.1, U$1.GND, U$2.GND; no longer C1.2, C10.2, C12.1, C13.1, C14.1, C16.2, C17.1, C18.2, C2.2, C20.2, C21.2, C23.2, C24.2, C25.2, C26.2, C27.2, C28.2, C29.2, C3.2, C30.2, C32.2, C4.2, C5.2, C6.2, C7.2, C8.1, C9.1, G1.-, IC2.!RST, IC2.GND, IC2.NC@0, IC2.NC@1, IC2.NC@2, IC2.NC@3, IC2.NC@4, IC2.NC@5, IC2.NC@6, IC2.NC@7, J2.GND@0, J2.GND@1, R11.2, R14.2, R15.2, R18.1, R24.2, R35.2, R4.2, R6.2, T1.E, T2.E, T4.E, TP1.TP, TP101.TP, U$1.10, U$1.12, U$1.27, U$1.37, U$1.39, U$1.41, U$1.44, U$17.A1, U$17.A2, U$17.GND, U$3.GND, U$3.SH@1, U$3.SH@2, U$3.SH@3, U$3.SH@4, U$6G$1.EN1, U$6G$1.TD, U$6G$1.VSS, U$6TH.TH, U$8.ANODE, U1.GND, U3.GND, X1.6, X2.2, X4.1, X6.4
- net SCL_H: now also R5.1; no longer Q2.D, R10.1
- net SDA_H: now also R7.1; no longer Q3.D, R2.1
Other:
- note removed: "ILIM=1610/R15"
- note removed: "ISET=890/R11"
- note removed: "digital input pins: - RI (detect incoming sms) - CTS - ^CH (LiPo charging)"
- note removed: "digital output pins: - CE (LiPo charge enable) - 3V3_EN - GPRS_EN - GPRS_POW - VBACKUP (GPS) - PW_EN - DTR (wake up gprs) - RTS"
- note removed: "uC pins: 7 11 28"
- moved on the sheet: C1, C2, C7, R13

Commit message: pcb verified
Parts:
- removed C7: 100nF, rcl:C-EUC0805
Connections:
- net +3V3: no longer C7.2
- net GND: no longer C7.1
Other:
- moved on the sheet: C1, C15, C2, R13, R5, R7, R8, U$1, X5
